File: docs/kicad/board/combined.kicad_pcb (KiCad board)
At the start: 2 copper layers, 64 x 84 mm, 29 parts, among them J1 G 5 L D, J1 VIN, J10 WHEEL_4, J11 FLAG, J12 LED, J13 COMPASS, J14 SWITCH, J2 LEFT, J3 CENTER, J4 RIGHT, J5 ARM, J6 LID, J7 WHEEL_1, J8 WHEEL_2, J9 WHEEL_3, SW1 BUTTON_1, SW2 BUTTON_2, U1 ARDUINO_NANO

Commit message: Built version 2 for Daniel
Parts:
- removed J4: RIGHT, cnc3018-PCB:my4pin
- J3: value CENTER -> RIGHT
- moved U1 0.06 mm to (41.9, -32.5)
- moved J10 0.06 mm to (42.4, -14.7)
- moved J11 0.06 mm to (44.9, -14.7)
- moved J6 0.06 mm to (32.2, -14.7)
- moved J8 0.06 mm to (37.3, -14.7)
- moved J9 0.06 mm to (39.8, -14.7)
- moved J13 0.06 mm to (11.4, -4.58)
- moved J14 0.06 mm to (16.5, -12.2)
- moved J5 0.06 mm to (29.6, -14.7)
- moved J12 0.06 mm to (6.32, -12.2)
- moved J1 0.06 mm to (19.0, -50.3)
- moved J2 0.06 mm to (26.6, -50.3)
- moved J3 0.06 mm to (39.3, -50.3)
- moved J7 0.06 mm to (34.7, -14.7)
- moved SW1 0.06 mm to (59.7, -8.39)
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Connections:
- J2 pad 3: L_SENS -> L_IR
- J2 pad 4: L_IR -> L_SENS
- J3 pad 3: C_SENS -> R_IR
- J3 pad 4: C_IR -> R_SENS
- U1 pad 10: C_IR -> R_SENS
- U1 pad 11: Net-(U1-Pad11) -> L_IR
- U1 pad 13: R_SENS -> Net-(U1-Pad13)
- U1 pad 15: R_IR -> Net-(U1-Pad15)
- U1 pad 5: L_SENS -> Net-(U1-Pad5)
- U1 pad 6: L_IR -> L_SENS
- U1 pad 9: C_SENS -> R_IR
Routing:
- net +5V: track 90.4 -> 72.6 mm, vias 4 -> 2
- net L_IR: track 11.2 -> 27.0 mm, vias 0 -> 2
- net C_SENS: track 10.2 -> 0.00 mm
- net C_IR: track 10.2 -> 0.00 mm
- net R_SENS: track 11.2 -> 10.2 mm
Other:
- outline, holes or cut-outs redrawn
